Commit message: Complete version with Isaac Sim data collection

File: T170A/urdf/T170A.urdf (robot description, URDF)
Before this commit: robot T170A, 59 links, 58 joints
Joints:
- joint left_elbow_pitch: limit lower=-1.92 upper=0 effort=34 velocity=3.87 -> lower=-2.06 upper=0 effort=34 velocity=3.87
- joint right_elbow_pitch: limit lower=0 upper=1.92 effort=34 velocity=3.87 -> lower=0 upper=2.06 effort=34 velocity=3.87
